Commit message: added 3d_lidar and depth camera for stvl

File: description/round_bot_with_depth_camera_and_3d_lidar.urdf.xacro (robot description, xacro)
@@ -196,5 +196,5 @@
   <link name="camera_link_optical">
   </link>
-  <!-- camera -->
+  <!-- depth camera -->
   <gazebo reference="camera_link">
     <material>Gazebo/Blue</material>
@@ -246,9 +246,9 @@
   </joint>
   <!-- 3d lidar -->
-  <!-- <gazebo reference="lidar_link">
-    <material>Gazebo/Red</material>
-    <sensor type="ray" name="block_laser_sensor">
+  <gazebo reference="lidar_link">
+    <material>Gazebo/Red</material>
+    <sensor type="ray" name="3d_lidar">
       <pose>0 0 0 0 0 0</pose>
-      <visualize>false</visualize>
+      <visualize>true</visualize>
       <ray>
         <scan>
@@ -272,5 +272,5 @@
         </range>
       </ray>
-      <plugin name="gazebo_ros_block_laser_controller" filename="libgazebo_ros_ray_sensor.so">
+      <plugin name="gazebo_ros_block_laser_controller_1" filename="libgazebo_ros_velodyne_laser.so">
         <ros>
           <remapping>~/out:=velodyne_points</remapping>
@@ -285,14 +285,14 @@
         <output_type>sensor_msgs/PointCloud2</output_type>
         <alwaysOn>true</alwaysOn>
-        <updateRate>1</updateRate>
+        <updateRate>10</updateRate>
         <topicName>velodyne_points</topicName>
         <frame_name>lidar_link</frame_name>
       </plugin>
     </sensor>
-  </gazebo> -->
+  </gazebo>
   <!-- 2d lidar -->
   <gazebo reference="lidar_link">
     <material>Gazebo/Red</material>
-      <sensor name="block_laser_sensor" type="ray">
+      <sensor name="2d_lidar" type="ray">
       <pose> 0 0 0 0 0 0 </pose>
       <visualize>true</visualize>
@@ -318,5 +318,5 @@
         </noise>
       </ray>
-      <plugin name="gazebo_ros_block_laser_controller" filename="libgazebo_ros_ray_sensor.so">
+      <plugin name="gazebo_ros_block_laser_controller_2" filename="libgazebo_ros_ray_sensor.so">
         <ros>
           <remapping>~/out:=scan</remapping>
