Commit message: world is created and robot moves

File: description/inertial_xacros.xacro (robot description, xacro)
@@ -5,8 +5,8 @@
     <xacro:property name="wheel_radius" value="0.08"/>
     <xacro:property name="wheel_length" value="0.05"/>
-    <xacro:property name="wheel_mass" value="0.1"/>
+    <xacro:property name="wheel_mass" value="0.75"/>
     <xacro:property name="chassis_radius" value="0.35"/>
     <xacro:property name="chassis_length" value="0.1"/>
-    <xacro:property name="chassis_mass" value="0.5"/>
+    <xacro:property name="chassis_mass" value="2"/>
     <xacro:property name="mount_radius" value="0.08"/>
     <xacro:property name="mount_length" value="0.05"/>
@@ -15,5 +15,5 @@
     <xacro:property name="lidar_length" value="0.07"/>
     <xacro:property name="lidar_mass" value="0.1"/>
-    <xacro:property name="caster_mass" value="0.1"/>
+    <xacro:property name="caster_mass" value="0.75"/>
     <xacro:property name="caster_radius" value="0.05"/>
     <xacro:macro name="inertial_sphere" params="caster_mass caster_radius *origin">

File: description/round_bot.urdf.xacro (robot description, xacro)
@@ -2,6 +2,5 @@
 <robot xmlns:xacro="http://www.ros.org/wiki/xacro" name="round_bot">
 <xacro:include filename="$(find round_bot)/description/inertial_xacros.xacro"/>
-  <link name="base_link">
-  </link>
+  <link name="base_link"/>
   <joint name="chassis_joint" type="fixed">
     <parent link="base_link"/>
@@ -13,5 +12,4 @@
       <origin xyz="0.0 0.0 0.12" rpy="0.0 0.0 0.0"/>
       <geometry>
-        <!-- <cylinder radius="0.35" length="0.1"/> -->
         <cylinder radius="${chassis_radius}" length="${chassis_length}"/>
       </geometry>
@@ -23,8 +21,7 @@
       <origin xyz="0.0 0.0 0.12" rpy="0.0 0.0 0.0"/>
       <geometry>
-          <!-- <sphere radius="0.0"/> -->
-          <cylinder radius="${chassis_radius}" length="${chassis_length}"/>
-          <!-- <contact_coefficients mu = "1" kp = "1e+13" kd = "1.0"/> -->
-      </geometry>
+        <cylinder radius="${chassis_radius}" length="${chassis_length}"/>
+      </geometry>
+      <contact_coefficients mu1 = "1" mu2 = "1" kp = "1e+13.0" kd = "1.0"/>
     </collision>
     <xacro:inertial_chassis_cylinder chassis_mass="${chassis_mass}" chassis_length="${chassis_length}" chassis_radius="${chassis_radius}">
@@ -54,6 +51,6 @@
       <geometry>
         <sphere radius="${wheel_radius}"/>
-        <contact_coefficients mu = "1" kp = "1e+13" kd = "1.0"/>
-      </geometry>
+      </geometry>
+      <contact_coefficients mu1 = "0" kp = "1000.0" kd = "1.0"/>
     </collision>
     <xacro:inertial_wheel_cylinder wheel_mass="${wheel_mass}" wheel_length="${wheel_length}" wheel_radius="${wheel_radius}">
@@ -62,10 +59,4 @@
   </link>
   <gazebo reference = "left_wheel">
-      <mu1 value="50"/>
-      <mu2 value="50"/>
-      <kp value="1000000.0" />
-      <kd value="100.0" />
-      <slip1 value="0.5" />
-      <slip2 value="0.5" />
     <material>Gazebo/Red</material>
   </gazebo>
@@ -89,6 +80,6 @@
       <geometry>
         <sphere radius="${wheel_radius}"/>
-        <contact_coefficients mu = "1" kp = "1e+13" kd = "1.0"/>
-      </geometry>
+      </geometry>
+      <contact_coefficients mu = "0" kp = "1000.0" kd = "1.0"/>
     </collision>
     <xacro:inertial_wheel_cylinder wheel_mass="${wheel_mass}" wheel_length="${wheel_length}" wheel_radius="${wheel_radius}">
@@ -97,10 +88,6 @@
   </link>
   <gazebo reference = "right_wheel">
-      <mu1 value="100"/>
-      <mu2 value="100"/>
-      <kp value="1000000.0" />
-      <kd value="100.0" />
-      <slip1 value="0.5" />
-      <slip2 value="0.5" />
+    <slip1 value="0.5" />
+    <slip2 value="0.5" />
     <material>Gazebo/Red</material>
   </gazebo>
@@ -108,5 +95,5 @@
     <parent link="chassis"/>
     <child link="front_caster_link"/>
-    <origin xyz="0.25 0.0 0.04" rpy="0 0 0"/>
+    <origin xyz="0.25 0.0 0.0465" rpy="0 0 0"/>
     <mu1 value="0.001"/>
     <mu2 value="0.001"/>
@@ -126,4 +113,5 @@
         <sphere radius="${caster_radius}"/>
       </geometry>
+      <contact_coefficients mu="0" kp="1000.0" kd="1.0"/>
     </collision>
     <xacro:inertial_sphere caster_mass="${caster_mass}" caster_radius="${caster_radius}">
@@ -137,5 +125,5 @@
     <parent link="chassis"/>
     <child link="back_caster_link"/>
-    <origin xyz="-0.25 0.0 0.04" rpy="0 0 0"/>
+    <origin xyz="-0.25 0.0 0.0465" rpy="0 0 0"/>
     <mu1 value="0.001"/>
     <mu2 value="0.001"/>
@@ -155,4 +143,5 @@
         <sphere radius="${caster_radius}"/>
       </geometry>
+      <contact_coefficients mu="0" kp="1000.0" kd="1.0"/>
     </collision>
     <xacro:inertial_sphere caster_mass="${caster_mass}" caster_radius="${caster_radius}">

Commit message: implemented slam, localization and navigation, reduced the bot chassis radius

File: description/inertial_xacros.xacro (robot description, xacro)
@@ -6,5 +6,5 @@
     <xacro:property name="wheel_length" value="0.05"/>
     <xacro:property name="wheel_mass" value="0.75"/>
-    <xacro:property name="chassis_radius" value="0.35"/>
+    <xacro:property name="chassis_radius" value="0.25"/>
     <xacro:property name="chassis_length" value="0.1"/>
     <xacro:property name="chassis_mass" value="2"/>

File: description/round_bot.urdf.xacro (robot description, xacro)
@@ -1,8 +1,9 @@
 <?xml version="1.0"?>
 <robot xmlns:xacro="http://www.ros.org/wiki/xacro" name="round_bot">
-<xacro:include filename="$(find round_bot)/description/inertial_xacros.xacro"/>
-  <link name="base_link"/>
+  <xacro:include filename="$(find round_bot)/description/inertial_xacros.xacro"/>
+  <!-- <xacro:include filename="$(find round_bot)/description/ros2_control.xacro"/> -->
+  <link name="base_footprint"/>
   <joint name="chassis_joint" type="fixed">
-    <parent link="base_link"/>
+    <parent link="base_footprint"/>
     <child link="chassis"/>
     <origin xyz="0.0 0.0 0.0" rpy="0.0 0.0 0.0"/>
@@ -36,5 +37,5 @@
     <child link="left_wheel"/>
     <axis xyz="0 0 1.0"/>
-    <origin xyz="0.0 0.25 0.075" rpy="-1.57 0.0 0.0"/>
+    <origin xyz="0.0 0.18 0.075" rpy="-1.57 0.0 0.0"/>
   </joint>
   <link name="left_wheel">
@@ -65,5 +66,5 @@
     <child link="right_wheel"/>
     <axis xyz="0.0 0.0 1.0"/>
-    <origin xyz="0.0 -0.25 0.075" rpy="-1.57 0.0 0.0"/>
+    <origin xyz="0.0 -0.18 0.075" rpy="-1.57 0.0 0.0"/>
   </joint>
   <link name="right_wheel">
@@ -95,5 +96,5 @@
     <parent link="chassis"/>
     <child link="front_caster_link"/>
-    <origin xyz="0.25 0.0 0.0465" rpy="0 0 0"/>
+    <origin xyz="0.18 0.0 0.0452" rpy="0 0 0"/>
     <mu1 value="0.001"/>
     <mu2 value="0.001"/>
@@ -125,5 +126,5 @@
     <parent link="chassis"/>
     <child link="back_caster_link"/>
-    <origin xyz="-0.25 0.0 0.0465" rpy="0 0 0"/>
+    <origin xyz="-0.18 0.0 0.0452" rpy="0 0 0"/>
     <mu1 value="0.001"/>
     <mu2 value="0.001"/>
@@ -155,5 +156,5 @@
     <parent link="chassis"/>
     <child link="mount_link"/>
-    <origin xyz="0.2 0.0 0.2" rpy="0.0 0.0 0.0"/>
+    <origin xyz="0.15 0.0 0.2" rpy="0.0 0.0 0.0"/>
   </joint>
   <link name="mount_link">
@@ -190,5 +191,5 @@
   </link>
   <joint name="camera_joint" type="fixed">
-    <origin xyz="0.35 0.0 0.125" rpy="0 0 0"/>
+    <origin xyz="0.25 0.0 0.125" rpy="0 0 0"/>
     <parent link="chassis"/>
     <child link="camera_link"/>
@@ -219,5 +220,5 @@
       </camera>
       <plugin name="camera_controller" filename="libgazebo_ros_camera.so">
-        <!-- <alwaysOn>true</alwaysOn> -->
+        <alwaysOn>true</alwaysOn>
         <frameName>camera_link_optical</frameName>
       </plugin>
@@ -266,5 +267,5 @@
         <range>
           <min>0.3</min>
-          <max>15.0</max>
+          <max>5.0</max>
           <resolution>0.1</resolution>
         </range>
@@ -284,24 +285,4 @@
     </sensor>
   </gazebo>
-  <transmission name="left_wheel_transmission">
-    <type>transmission_interface/SimpleTransmission</type>
-    <joint name="left_wheel_joint">
-      <hardwareInterface>hardware_interface/VelocityJointInterface</hardwareInterface>
-    </joint>
-    <actuator name="left_wheel_motor">
-      <mechanicalReduction>1</mechanicalReduction>
-      <hardwareInterface>hardware_interface/VelocityJointInterface</hardwareInterface>
-    </actuator>
-  </transmission>
-  <transmission name="right_wheel_transmission">
-    <type>transmission_interface/SimpleTransmission</type>
-    <joint name="right_wheel_joint">
-      <hardwareInterface>hardware_interface/VelocityJointInterface</hardwareInterface>
-    </joint>
-    <actuator name="right_wheel_motor">
-      <mechanicalReduction>1</mechanicalReduction>
-      <hardwareInterface>hardware_interface/VelocityJointInterface</hardwareInterface>
-    </actuator>
-  </transmission>
   <gazebo>
     <plugin name='diff_drive' filename='libgazebo_ros_diff_drive.so'>
@@ -309,5 +290,5 @@
       <left_joint>left_wheel_joint</left_joint>
       <right_joint>right_wheel_joint</right_joint>
-      <wheel_separation>0.50</wheel_separation>
+      <wheel_separation>0.36</wheel_separation>
       <wheel_diameter>0.16</wheel_diameter>
       <max_wheel_torque>10</max_wheel_torque>
@@ -318,5 +299,5 @@
       <odometry_source>1</odometry_source>
       <odometry_frame>odom</odometry_frame>
-      <robot_base_frame>base_link</robot_base_frame>
+      <robot_base_frame>base_footprint</robot_base_frame>
     </plugin>
   </gazebo>

Commit message: launch log file added

File: description/inertial_xacros.xacro (robot description, xacro)
@@ -9,9 +9,9 @@
     <xacro:property name="chassis_length" value="0.1"/>
     <xacro:property name="chassis_mass" value="2"/>
-    <xacro:property name="mount_radius" value="0.08"/>
-    <xacro:property name="mount_length" value="0.05"/>
+    <xacro:property name="mount_radius" value="0.04"/>
+    <xacro:property name="mount_length" value="0.04"/>
     <xacro:property name="mount_mass" value="0.1"/>
-    <xacro:property name="lidar_radius" value="0.1"/>
-    <xacro:property name="lidar_length" value="0.07"/>
+    <xacro:property name="lidar_radius" value="0.07"/>
+    <xacro:property name="lidar_length" value="0.04"/>
     <xacro:property name="lidar_mass" value="0.1"/>
     <xacro:property name="caster_mass" value="0.75"/>

File: description/round_bot.urdf.xacro (robot description, xacro)
@@ -156,5 +156,5 @@
     <parent link="chassis"/>
     <child link="mount_link"/>
-    <origin xyz="0.15 0.0 0.2" rpy="0.0 0.0 0.0"/>
+    <origin xyz="0.15 0.0 0.18" rpy="0.0 0.0 0.0"/>
   </joint>
   <link name="mount_link">
@@ -246,5 +246,5 @@
   </link>
   <joint name="lidar_joint" type="fixed">
-    <origin xyz="0.0 0 0.05" rpy="0 0.0 0.0"/>
+    <origin xyz="0.0 0 0.03" rpy="0 0.0 0.0"/>
     <parent link="mount_link"/>
     <child link="lidar_link"/>
