Commit message: initial commit for new gazebo

File: description/inertial_xacros.xacro (robot description, xacro)
@@ -1,73 +1,64 @@
 <?xml version="1.0"?>
 <robot xmlns:xacro="http://www.ros.org/wiki/xacro" name="round_bot">
-    <!-- Specify some standard inertial calculations https://en.wikipedia.org/wiki/List_of_moments_of_inertia -->
-    <!-- These make use of xacro's mathematical functionality -->
-    <xacro:property name="wheel_radius" value="0.08"/>
-    <xacro:property name="wheel_length" value="0.05"/>
-    <xacro:property name="wheel_mass" value="0.75"/>
-    <xacro:property name="chassis_radius" value="0.25"/>
-    <xacro:property name="chassis_length" value="0.1"/>
-    <xacro:property name="chassis_mass" value="2"/>
-    <xacro:property name="mount_radius" value="0.04"/>
-    <xacro:property name="mount_length" value="0.04"/>
-    <xacro:property name="mount_mass" value="0.1"/>
-    <xacro:property name="lidar_radius" value="0.07"/>
-    <xacro:property name="lidar_length" value="0.04"/>
-    <xacro:property name="lidar_mass" value="0.1"/>
-    <xacro:property name="caster_mass" value="0.75"/>
-    <xacro:property name="caster_radius" value="0.05"/>
-    <xacro:macro name="inertial_sphere" params="caster_mass caster_radius *origin">
-        <inertial>
-            <xacro:insert_block name="origin"/>
-            <mass value="${caster_mass}" />
-            <inertia ixx="${(2/5) * caster_mass * (caster_radius*caster_radius)}" ixy="0.0" ixz="0.0"
-                    iyy="${(2/5) * caster_mass * (caster_radius*caster_radius)}" iyz="0.0"
-                    izz="${(2/5) * caster_mass * (caster_radius*caster_radius)}" />
-        </inertial>
-    </xacro:macro>
-    <!-- <xacro:macro name="inertial_box" params="mass x y z *origin">
-        <inertial>
-            <xacro:insert_block name="origin"/>
-            <mass value="${mass}" />
-            <inertia ixx="${(1/12) * mass * (y*y+z*z)}" ixy="0.0" ixz="0.0"
-                    iyy="${(1/12) * mass * (x*x+z*z)}" iyz="0.0"
-                    izz="${(1/12) * mass * (x*x+y*y)}" />
-        </inertial>
-    </xacro:macro> -->
-    <xacro:macro name="inertial_wheel_cylinder" params="wheel_mass wheel_length wheel_radius *origin">
-        <inertial>
-            <xacro:insert_block name="origin"/>
-            <mass value="${wheel_mass}" />
-            <inertia ixx="${(1/12) * wheel_mass * (3*wheel_radius*wheel_radius + wheel_length*wheel_length)}" ixy="0.0" ixz="0.0"
-                    iyy="${(1/12) * wheel_mass * (3*wheel_radius*wheel_radius + wheel_length*wheel_length)}" iyz="0.0"
-                    izz="${(1/2) * wheel_mass * (wheel_radius*wheel_radius)}" />
-        </inertial>
-    </xacro:macro>
-    <xacro:macro name="inertial_chassis_cylinder" params="chassis_mass chassis_length chassis_radius *origin">
-        <inertial>
-            <xacro:insert_block name="origin"/>
-            <mass value="${chassis_mass}" />
-            <inertia ixx="${(1/12) * chassis_mass * (3*chassis_radius*chassis_radius + chassis_length*chassis_length)}" ixy="0.0" ixz="0.0"
-                    iyy="${(1/12) * chassis_mass * (3*chassis_radius*chassis_radius + chassis_length*chassis_length)}" iyz="0.0"
-                    izz="${(1/2) * chassis_mass * (chassis_radius*chassis_radius)}" />
-        </inertial>
-    </xacro:macro>
-    <xacro:macro name="inertial_mount_cylinder" params="mount_mass mount_length mount_radius *origin">
-        <inertial>
-            <xacro:insert_block name="origin"/>
-            <mass value="${mount_mass}" />
-            <inertia ixx="${(1/12) * mount_mass * (3*mount_radius*mount_radius + mount_length*mount_length)}" ixy="0.0" ixz="0.0"
-                    iyy="${(1/12) * mount_mass * (3*mount_radius*mount_radius + mount_length*mount_length)}" iyz="0.0"
-                    izz="${(1/2) * mount_mass * (mount_radius*mount_radius)}" />
-        </inertial>
-    </xacro:macro>
-    <xacro:macro name="inertial_lidar_cylinder" params="lidar_mass lidar_length lidar_radius *origin">
-        <inertial>
-            <xacro:insert_block name="origin"/>
-            <mass value="${lidar_mass}" />
-            <inertia ixx="${(1/12) * lidar_mass * (3*lidar_radius*lidar_radius + lidar_length*lidar_length)}" ixy="0.0" ixz="0.0"
-                    iyy="${(1/12) * lidar_mass * (3*lidar_radius*lidar_radius + lidar_length*lidar_length)}" iyz="0.0"
-                    izz="${(1/2) * lidar_radius * (lidar_radius*lidar_radius)}" />
-        </inertial>
-    </xacro:macro>
+	<!-- Specify some standard inertial calculations https://en.wikipedia.org/wiki/List_of_moments_of_inertia -->
+	<!-- These make use of xacro's mathematical functionality -->
+	<xacro:property name="wheel_radius" value="0.08"/>
+	<xacro:property name="wheel_length" value="0.05"/>
+	<xacro:property name="wheel_mass" value="0.75"/>
+	<xacro:property name="chassis_radius" value="0.25"/>
+	<xacro:property name="chassis_length" value="0.1"/>
+	<xacro:property name="chassis_mass" value="2"/>
+	<xacro:property name="mount_radius" value="0.04"/>
+	<xacro:property name="mount_length" value="0.04"/>
+	<xacro:property name="mount_mass" value="0.1"/>
+	<xacro:property name="lidar_radius" value="0.07"/>
+	<xacro:property name="lidar_length" value="0.04"/>
+	<xacro:property name="lidar_mass" value="0.1"/>
+	<xacro:property name="caster_mass" value="0.75"/>
+	<xacro:property name="caster_radius" value="0.05"/>
+	<xacro:macro name="inertial_sphere" params="caster_mass caster_radius *origin">
+		<inertial>
+			<xacro:insert_block name="origin"/>
+			<mass value="${caster_mass}" />
+			<inertia ixx="${(2/5) * caster_mass * (caster_radius*caster_radius)}" ixy="0.0" ixz="0.0"
+							iyy="${(2/5) * caster_mass * (caster_radius*caster_radius)}" iyz="0.0"
+							izz="${(2/5) * caster_mass * (caster_radius*caster_radius)}" />
+		</inertial>
+	</xacro:macro>
+	<xacro:macro name="inertial_wheel_cylinder" params="wheel_mass wheel_length wheel_radius *origin">
+		<inertial>
+			<xacro:insert_block name="origin"/>
+			<mass value="${wheel_mass}" />
+			<inertia ixx="${(1/12) * wheel_mass * (3*wheel_radius*wheel_radius + wheel_length*wheel_length)}" ixy="0.0" ixz="0.0"
+							iyy="${(1/12) * wheel_mass * (3*wheel_radius*wheel_radius + wheel_length*wheel_length)}" iyz="0.0"
+							izz="${(1/2) * wheel_mass * (wheel_radius*wheel_radius)}" />
+		</inertial>
+	</xacro:macro>
+	<xacro:macro name="inertial_chassis_cylinder" params="chassis_mass chassis_length chassis_radius *origin">
+		<inertial>
+			<xacro:insert_block name="origin"/>
+			<mass value="${chassis_mass}" />
+			<inertia ixx="${(1/12) * chassis_mass * (3*chassis_radius*chassis_radius + chassis_length*chassis_length)}" ixy="0.0" ixz="0.0"
+							iyy="${(1/12) * chassis_mass * (3*chassis_radius*chassis_radius + chassis_length*chassis_length)}" iyz="0.0"
+							izz="${(1/2) * chassis_mass * (chassis_radius*chassis_radius)}" />
+		</inertial>
+	</xacro:macro>
+	<xacro:macro name="inertial_mount_cylinder" params="mount_mass mount_length mount_radius *origin">
+		<inertial>
+			<xacro:insert_block name="origin"/>
+			<mass value="${mount_mass}" />
+			<inertia ixx="${(1/12) * mount_mass * (3*mount_radius*mount_radius + mount_length*mount_length)}" ixy="0.0" ixz="0.0"
+							iyy="${(1/12) * mount_mass * (3*mount_radius*mount_radius + mount_length*mount_length)}" iyz="0.0"
+							izz="${(1/2) * mount_mass * (mount_radius*mount_radius)}" />
+		</inertial>
+	</xacro:macro>
+	<xacro:macro name="inertial_lidar_cylinder" params="lidar_mass lidar_length lidar_radius *origin">
+		<inertial>
+			<xacro:insert_block name="origin"/>
+			<mass value="${lidar_mass}" />
+			<inertia ixx="${(1/12) * lidar_mass * (3*lidar_radius*lidar_radius + lidar_length*lidar_length)}" ixy="0.0" ixz="0.0"
+							iyy="${(1/12) * lidar_mass * (3*lidar_radius*lidar_radius + lidar_length*lidar_length)}" iyz="0.0"
+							izz="${(1/2) * lidar_radius * (lidar_radius*lidar_radius)}" />
+		</inertial>
+	</xacro:macro>
 </robot>

File: description/round_bot.urdf.xacro (robot description, xacro)
@@ -2,4 +2,5 @@
 <robot xmlns:xacro="http://www.ros.org/wiki/xacro" name="round_bot">
   <xacro:include filename="$(find round_bot)/description/inertial_xacros.xacro"/>
+  <xacro:property name="use_2d_lidar" value="true" />
   <link name="base_footprint"/>
   <joint name="chassis_joint" type="fixed">
@@ -49,7 +50,7 @@
     <collision>
       <geometry>
-        <sphere radius="${wheel_radius}"/>
-      </geometry>
-      <contact_coefficients mu1 = "0" kp = "1000.0" kd = "1.0"/>
+        <cylinder radius="${wheel_radius}" length="${wheel_length}"/>
+      </geometry>
+      <contact_coefficients mu1="1.0" mu2="1.0" kp="1000.0" kd="1.0"/>
     </collision>
     <xacro:inertial_wheel_cylinder wheel_mass="${wheel_mass}" wheel_length="${wheel_length}" wheel_radius="${wheel_radius}">
@@ -77,7 +78,7 @@
     <collision>
       <geometry>
-        <sphere radius="${wheel_radius}"/>
-      </geometry>
-      <contact_coefficients mu = "0" kp = "1000.0" kd = "1.0"/>
+        <cylinder radius="${wheel_radius}" length="${wheel_length}"/>
+      </geometry>
+      <contact_coefficients mu1="1.0" mu2="1.0" kp="1000.0" kd="1.0"/>
     </collision>
     <xacro:inertial_wheel_cylinder wheel_mass="${wheel_mass}" wheel_length="${wheel_length}" wheel_radius="${wheel_radius}">
@@ -86,6 +87,4 @@
   </link>
   <gazebo reference = "right_wheel">
-    <slip1 value="0.5" />
-    <slip2 value="0.5" />
     <material>Gazebo/Red</material>
   </gazebo>
@@ -148,5 +147,5 @@
     <material>Gazebo/Red</material>
   </gazebo>
-  <joint name="mount_joint" type="fixed">
+<!--  <joint name="mount_joint" type="fixed">
     <parent link="chassis"/>
     <child link="mount_link"/>
@@ -173,4 +172,44 @@
   <gazebo reference = "mount_link">
     <material>Gazebo/Black</material>
+  </gazebo> -->
+  <link name="imu_link">
+    <visual>
+      <origin xyz="0 0 0.0" rpy="0 0 0"/>
+      <geometry>
+        <box size="0.03 0.03 0.02"/>
+      </geometry>
+      <material name="green">
+        <color rgba="0 1 0 1"/>
+      </material>
+    </visual>
+    <collision>
+      <origin xyz="0 0 0.02" rpy="0 0 0"/>
+      <geometry>
+        <box size="0.03 0.03 0.02"/>
+      </geometry>
+    </collision>
+    <inertial>
+      <mass value="0.01"/>
+      <origin xyz="0 0 0.02" rpy="0 0 0"/>
+      <inertia ixx="1e-6" ixy="0" ixz="0" iyy="1e-6" iyz="0" izz="1e-6"/>
+    </inertial>
+  </link>
+  <joint name="imu_joint" type="fixed">
+    <parent link="chassis"/>
+    <child link="imu_link"/>
+    <origin xyz="0.0 0.0 0.165" rpy="0.0 0.0 0.0"/>
+  </joint>
+  <gazebo reference="imu_link">
+    <material>Gazebo/Green</material>
+    <sensor name="imu_sensor" type="imu">
+      <always_on>true</always_on>
+      <update_rate>100.0</update_rate>
+      <visualize>true</visualize>
+      <topic>imu</topic>
+      <gz_frame_id>imu_link</gz_frame_id>
+      <plugin name="gz::sim::systems::Imu" filename="gz-sim-imu-system">
+        <topic>imu</topic>
+      </plugin>
+    </sensor>
   </gazebo>
   <link name="camera_link">
@@ -198,8 +237,9 @@
   <!-- camera -->
   <gazebo reference="camera_link">
-    <material>Gazebo/Blue</material>
+    <material> Gazebo/Blue</material>
     <sensor type="camera" name="camera">
       <update_rate>10.0</update_rate>
       <camera name="head">
+        <camera_info_topic>camera/camera_info</camera_info_topic>
           <horizontal_fov>1.3962634</horizontal_fov>
           <image>
@@ -213,8 +253,6 @@
           </clip>
       </camera>
-      <plugin name="camera_controller" filename="libgazebo_ros_camera.so">
-        <alwaysOn>true</alwaysOn>
-        <frameName>camera_link_optical</frameName>
-      </plugin>
+      <topic>camera/image_raw</topic>
+      <gz_frame_id>camera_link_optical</gz_frame_id>
     </sensor>
   </gazebo>
@@ -238,59 +276,106 @@
   </link>
   <joint name="lidar_joint" type="fixed">
-    <origin xyz="0.0 0 0.03" rpy="0 0.0 0.0"/>
-    <parent link="mount_link"/>
+    <!-- <origin xyz="0.0 0.0 0.03" rpy="0.0 0.0 0.0"/>
+    <parent link="mount_link"/> -->
+    <origin xyz="0.15 0.0 0.18" rpy="0.0 0.0 0.0"/>
+    <parent link="chassis"/>
     <child link="lidar_link"/>
   </joint>
-  <gazebo reference="lidar_link">
-    <material>Gazebo/Red</material>
-      <sensor name="block_laser_sensor" type="ray">
-      <pose> 0 0 0 0 0 0 </pose>
-      <visualize>true</visualize>
-      <update_rate>10.0</update_rate>
-      <ray>
-        <scan>
-          <horizontal>
-            <samples>360</samples>
-            <resolution>1.000000</resolution>
-            <min_angle>-3.14159</min_angle>
-            <max_angle>3.14159</max_angle>
-          </horizontal>
-        </scan>
-        <range>
-          <min>0.3</min>
-          <max>2.5</max>
-          <resolution>0.1</resolution>
-        </range>
-        <noise>
-          <type>gaussian</type>
-          <mean>0.0</mean>
-          <stddev>0.01</stddev>
-        </noise>
-      </ray>
-      <plugin name="gazebo_ros_block_laser_controller" filename="libgazebo_ros_ray_sensor.so">
-        <ros>
-          <remapping>~/out:=scan</remapping>
-        </ros>
-        <output_type>sensor_msgs/LaserScan</output_type>
-        <frame_name>lidar_link</frame_name>
-      </plugin>
-    </sensor>
-  </gazebo>
+  <!-- 2d lidar  -->
+  <xacro:if value="$(arg use_2d_lidar)">
+    <gazebo reference="lidar_link">
+      <material>Gazebo/Red</material>
+      <sensor name="hls_lfcd_lds" type="gpu_lidar">
+        <pose> 0 0 0 0 0 0 </pose>
+        <always_on>true</always_on>
+        <update_rate>30.0</update_rate>
+        <lidar>
+          <scan>
+            <horizontal>
+              <samples>360</samples>
+              <resolution>1.000000</resolution>
+              <min_angle>-3.14159</min_angle>
+              <max_angle>3.14159</max_angle>
+            </horizontal>
+          </scan>
+          <range>
+            <min>0.1</min>
+            <max>7.5</max>
+            <resolution>0.1</resolution>
+          </range>
+          <noise>
+            <type>gaussian</type>
+            <mean>0.0</mean>
+            <stddev>0.01</stddev>
+          </noise>
+        </lidar>
+        <topic>scan</topic>
+        <gz_frame_id>lidar_link</gz_frame_id>
+      </sensor>
+    </gazebo>
+  </xacro:if>
+  <!-- 3d lidar -->
+  <xacro:unless value="$(arg use_2d_lidar)">
+    <gazebo reference="lidar_link">
+      <material>Gazebo/Red</material>
+      <sensor name="block_laser_sensor" type="gpu_lidar">
+        <pose>0 0 0 0 0 0</pose>
+        <visualize>true</visualize>
+        <update_rate>30.0</update_rate>
+        <lidar>
+          <scan>
+            <horizontal>
+              <samples>180</samples>
+              <resolution>1.000000</resolution>
+              <min_angle>-3.14159</min_angle>
+              <max_angle>3.14159</max_angle>
+            </horizontal>
+            <vertical>
+              <samples>16</samples>
+              <resolution>0.1</resolution>
+              <min_angle>-0.2618</min_angle>
+              <max_angle>0.2618</max_angle>
+            </vertical>
+          </scan>
+          <range>
+            <min>0.5</min>
+            <max>7.5</max>
+            <resolution>0.1</resolution>
+          </range>
+          <point_cloud>true</point_cloud>
+          <noise>
+            <type>gaussian</type>
+            <mean>0.0</mean>
+            <stddev>0.01</stddev>
+          </noise>
+        </lidar>
+        <topic>velodyne_points</topic>
+        <gz_frame_id>lidar_link</gz_frame_id>
+      </sensor>
+    </gazebo>
+  </xacro:unless>
   <gazebo>
-    <plugin name='diff_drive' filename='libgazebo_ros_diff_drive.so'>
-      <update_rate>10</update_rate>
+    <plugin name='gz::sim::systems::DiffDrive' filename='gz-sim-diff-drive-system'>
       <left_joint>left_wheel_joint</left_joint>
       <right_joint>right_wheel_joint</right_joint>
       <wheel_separation>0.36</wheel_separation>
-      <wheel_diameter>0.16</wheel_diameter>
-      <max_wheel_torque>10</max_wheel_torque>
-      <max_wheel_acceleration>1.0</max_wheel_acceleration>
-      <publish_odom>true</publish_odom>
-      <publish_odom_tf>true</publish_odom_tf>
-      <publish_wheel_tf>true</publish_wheel_tf>
-      <odometry_source>1</odometry_source>
-      <odometry_frame>odom</odometry_frame>
-      <robot_base_frame>base_footprint</robot_base_frame>
+      <wheel_radius>0.08</wheel_radius>
+      <!-- <max_wheel_torque>10</max_wheel_torque> -->
+      <max_linear_acceleration>1.0</max_linear_acceleration>
+      <!-- <max_angular_acceleration>1.0</max_angular_acceleration> -->
+      <frame_id>odom</frame_id>
+      <child_frame_id>base_footprint</child_frame_id>
+      <odom_topic>odom</odom_topic>
+      <odom_publisher_frequency>30</odom_publisher_frequency>
+      <tf_topic>/tf</tf_topic>
+      <topic>cmd_vel</topic>
     </plugin>
+    <plugin filename="gz-sim-joint-state-publisher-system"
+      name="gz::sim::systems::JointStatePublisher">
+      <topic>joint_states</topic>
+      <joint_name>left_wheel_joint</joint_name>
+      <joint_name>right_wheel_joint</joint_name>
+      <!-- <update_rate>50</update_rate> -->
+    </plugin>
   </gazebo>
 </robot>
