Commit message: redefined the program

File: description/round_bot.urdf.xacro (robot description, xacro)
@@ -1,4 +1,4 @@
 <?xml version="1.0"?>
-<robot xmlns:xacro="http://www.ros.org/wiki/xacro" name="rount_bot">
+<robot xmlns:xacro="http://www.ros.org/wiki/xacro" name="roun_bot">
 <xacro:include filename="$(find round_bot)/description/inertial_xacros.xacro"/>
   <link name="base_footprint">
@@ -35,8 +35,63 @@
     <material>Gazebo/Orange </material>
   </gazebo>
-  <gazebo reference = "front_caster_link">
+  <joint name="left_wheel_joint" type="continuous">
+    <parent link="base_link"/>
+    <child link="left_wheel"/>
+    <axis xyz="0 0 1.0"/>
+    <origin xyz="0.25 0 0.075" rpy="1.57 0 1.57"/>
+  </joint>
+  <link name="left_wheel">
+    <visual>
+      <geometry>
+        <!-- <cylinder radius="0.08" length="0.05"/> -->
+        <cylinder radius="${wheel_radius}" length="${wheel_length}"/>
+      </geometry>
+      <material name = "Red">
+        <color rgba = "1.0 0.0 0.0 1.0"/>
+      </material>
+    </visual>
+    <collision>
+      <geometry>
+        <sphere radius="${wheel_radius}"/>
+        <contact_coefficients mu = "1" kp = "1e+13" kd = "1.0"/>
+      </geometry>
+    </collision>
+    <xacro:inertial_wheel_cylinder wheel_mass="${wheel_mass}" wheel_length="${wheel_length}" wheel_radius="${wheel_radius}">
+      <origin xyz="0 0 0" rpy="0 0 0"/>
+    </xacro:inertial_wheel_cylinder>
+  </link>
+  <gazebo reference = "left_wheel">
     <material>Gazebo/Red</material>
   </gazebo>
-  <joint name="front_caster_joint" type="continuous">
+  <joint name="right_wheel_joint" type="continuous">
+    <parent link="base_link"/>
+    <child link="right_wheel"/>
+    <axis xyz="0 0 1.0"/>
+    <origin xyz="-0.25 0 0.075" rpy="1.57 0 1.57"/>
+  </joint>
+  <link name="right_wheel">
+    <visual>
+      <geometry>
+        <!-- <cylinder radius="0.08" length="0.05"/> -->
+        <cylinder radius="${wheel_radius}" length="${wheel_length}"/>
+      </geometry>
+      <material name = "Red">
+        <color rgba = "1.0 0.0 0.0 1.0"/>
+      </material>
+    </visual>
+    <collision>
+      <geometry>
+        <sphere radius="${wheel_radius}"/>
+        <contact_coefficients mu = "1" kp = "1e+13" kd = "1.0"/>
+      </geometry>
+    </collision>
+    <xacro:inertial_wheel_cylinder wheel_mass="${wheel_mass}" wheel_length="${wheel_length}" wheel_radius="${wheel_radius}">
+      <origin xyz="0 0 0" rpy="0 0 0"/>
+    </xacro:inertial_wheel_cylinder>
+  </link>
+  <gazebo reference = "right_wheel">
+    <material>Gazebo/Red</material>
+  </gazebo>
+  <joint name="front_caster_joint" type="fixed">
     <parent link="base_link"/>
     <child link="front_caster_link"/>
@@ -45,5 +100,5 @@
     <mu2 value="0.001"/>
   </joint>
-  <link name="back_caster_link">
+  <link name="front_caster_link">
     <visual>
       <geometry>
@@ -64,8 +119,8 @@
     </xacro:inertial_sphere>
   </link>
-  <gazebo reference = "back_caster_link">
+  <gazebo reference = "front_caster_link">
     <material>Gazebo/Red</material>
   </gazebo>
-  <joint name="back_caster_joint" type="continuous">
+  <joint name="back_caster_joint" type="fixed">
     <parent link="base_link"/>
     <child link="back_caster_link"/>
@@ -74,5 +129,5 @@
     <mu2 value="0.001"/>
   </joint>
-  <link name="front_caster_link">
+  <link name="back_caster_link">
     <visual>
       <geometry>
@@ -93,62 +148,12 @@
     </xacro:inertial_sphere>
   </link>
-  <link name="left_wheel">
-    <visual>
-      <geometry>
-        <!-- <cylinder radius="0.08" length="0.05"/> -->
-        <cylinder radius="${wheel_radius}" length="${wheel_length}"/>
-      </geometry>
-      <material name = "Red">
-        <color rgba = "1.0 0.0 0.0 1.0"/>
-      </material>
-    </visual>
-    <collision>
-      <geometry>
-        <sphere radius="${wheel_radius}"/>
-        <contact_coefficients mu = "1" kp = "1e+13" kd = "1.0"/>
-      </geometry>
-    </collision>
-    <xacro:inertial_wheel_cylinder wheel_mass="${wheel_mass}" wheel_length="${wheel_length}" wheel_radius="${wheel_radius}">
-      <origin xyz="0 0 0" rpy="0 0 0"/>
-    </xacro:inertial_wheel_cylinder>
-  </link>
-  <joint name="left_wheel_joint" type="continuous">
-    <parent link="base_link"/>
-    <child link="left_wheel"/>
-    <axis xyz="0 0 1.0"/>
-    <origin xyz="0.25 0 0.075" rpy="1.57 0 1.57"/>
-  </joint>
-  <gazebo reference = "left_wheel">
+  <gazebo reference = "back_caster_link">
     <material>Gazebo/Red</material>
   </gazebo>
-  <link name="right_wheel">
-    <visual>
-      <geometry>
-        <!-- <cylinder radius="0.08" length="0.05"/> -->
-        <cylinder radius="${wheel_radius}" length="${wheel_length}"/>
-      </geometry>
-      <material name = "Red">
-        <color rgba = "1.0 0.0 0.0 1.0"/>
-      </material>
-    </visual>
-    <collision>
-      <geometry>
-        <sphere radius="${wheel_radius}"/>
-        <contact_coefficients mu = "1" kp = "1e+13" kd = "1.0"/>
-      </geometry>
-    </collision>
-    <xacro:inertial_wheel_cylinder wheel_mass="${wheel_mass}" wheel_length="${wheel_length}" wheel_radius="${wheel_radius}">
-      <origin xyz="0 0 0" rpy="0 0 0"/>
-    </xacro:inertial_wheel_cylinder>
-  </link>
-  <joint name="right_wheel_joint" type="continuous">
-    <parent link="base_link"/>
-    <child link="right_wheel"/>
-    <axis xyz="0 0 1.0"/>
-    <origin xyz="-0.25 0 0.075" rpy="1.57 0 1.57"/>
-  </joint>
-  <gazebo reference = "right_wheel">
-    <material>Gazebo/Red</material>
-  </gazebo>
+  <joint name="mount_joint" type="fixed">
+    <parent link="base_link"/>
+    <child link="mount_link"/>
+    <origin xyz="0.0 -0.2 0.2" rpy="0.0 0.0 0.0"/>
+  </joint>
   <link name="mount_link">
     <visual>
@@ -173,9 +178,4 @@
     <material>Gazebo/Black</material>
   </gazebo>
-  <joint name="mount_joint" type="fixed">
-    <parent link="base_link"/>
-    <child link="mount_link"/>
-    <origin xyz="0.0 -0.2 0.2" rpy="0.0 0.0 0.0"/>
-  </joint>
   <link name="camera_link">
     <visual>
@@ -303,30 +303,20 @@
     </actuator>
   </transmission>
-  <ros2_control name="GazeboSystem" type="system">
-    <hardware>
-        <plugin>gazebo_ros2_control/GazeboSystem</plugin>
-    </hardware>
-    <joint name="left_wheel_joint">
-      <command_interface name="velocity">
-        <param name="min">-10</param>
-        <param name="max">10</param>
-      </command_interface>
-      <state_interface name="velocity"/>
-      <state_interface name="position"/>
-    </joint>
-    <joint name="right_wheel_joint">
-      <command_interface name="velocity">
-        <param name="min">-10</param>
-        <param name="max">10</param>
-      </command_interface>
-      <state_interface name="velocity"/>
-      <state_interface name="position"/>
-    </joint>
-  </ros2_control>
   <gazebo>
-      <plugin name = "gazebo_ros2_control" filename="libgazebo_ros2_control.so">
-        <parameters>$(find round_bot)/config/control.yaml</parameters>
-        <!-- <robotNamespace></robotNamespace> -->
-      </plugin>
+    <plugin name='diff_drive' filename='libgazebo_ros_diff_drive.so'>
+      <update_rate>30</update_rate>
+      <left_joint>left_wheel_joint</left_joint>
+      <right_joint>right_wheel_joint</right_joint>\
+      <wheel_separation>0.50</wheel_separation>
+      <wheel_diameter>0.3</wheel_diameter>
+      <max_wheel_torque>10</max_wheel_torque>
+      <max_wheel_acceleration>1.0</max_wheel_acceleration>
+      <publish_odom>true</publish_odom>
+      <publish_odom_tf>true</publish_odom_tf>
+      <publish_wheel_tf>true</publish_wheel_tf>
+      <odometry_source>odom</odometry_source>
+      <odometry_frame>odom</odometry_frame>
+      <robot_base_frame>base_footprint</robot_base_frame>
+    </plugin>
   </gazebo>
 </robot>

Commit message: urdf changed

File: description/round_bot.urdf.xacro (robot description, xacro)
@@ -1,13 +1,13 @@
 <?xml version="1.0"?>
-<robot xmlns:xacro="http://www.ros.org/wiki/xacro" name="roun_bot">
+<robot xmlns:xacro="http://www.ros.org/wiki/xacro" name="round_bot">
 <xacro:include filename="$(find round_bot)/description/inertial_xacros.xacro"/>
-  <link name="base_footprint">
-  </link>
-  <joint name="base_link_joint" type="fixed">
-    <parent link="base_footprint"/>
-    <child link="base_link"/>
+  <link name="base_link">
+  </link>
+  <joint name="chassis_joint" type="fixed">
+    <parent link="base_link"/>
+    <child link="chassis"/>
     <origin xyz="0.0 0.0 0.0" rpy="0.0 0.0 0.0"/>
   </joint>
-  <link name="base_link">
+  <link name="chassis">
     <visual>
       <origin xyz="0.0 0.0 0.12" rpy="0.0 0.0 0.0"/>
@@ -32,12 +32,12 @@
     </xacro:inertial_chassis_cylinder>
   </link>
-  <gazebo reference = "base_link">
+  <gazebo reference = "chassis">
     <material>Gazebo/Orange </material>
   </gazebo>
   <joint name="left_wheel_joint" type="continuous">
-    <parent link="base_link"/>
+    <parent link="chassis"/>
     <child link="left_wheel"/>
     <axis xyz="0 0 1.0"/>
-    <origin xyz="0.25 0 0.075" rpy="1.57 0 1.57"/>
+    <origin xyz="0.0 0.25 0.075" rpy="-1.57 0.0 0.0"/>
   </joint>
   <link name="left_wheel">
@@ -62,11 +62,17 @@
   </link>
   <gazebo reference = "left_wheel">
+      <mu1 value="50"/>
+      <mu2 value="50"/>
+      <kp value="1000000.0" />
+      <kd value="100.0" />
+      <slip1 value="0.5" />
+      <slip2 value="0.5" />
     <material>Gazebo/Red</material>
   </gazebo>
   <joint name="right_wheel_joint" type="continuous">
-    <parent link="base_link"/>
+    <parent link="chassis"/>
     <child link="right_wheel"/>
-    <axis xyz="0 0 1.0"/>
-    <origin xyz="-0.25 0 0.075" rpy="1.57 0 1.57"/>
+    <axis xyz="0.0 0.0 1.0"/>
+    <origin xyz="0.0 -0.25 0.075" rpy="-1.57 0.0 0.0"/>
   </joint>
   <link name="right_wheel">
@@ -91,10 +97,16 @@
   </link>
   <gazebo reference = "right_wheel">
+      <mu1 value="100"/>
+      <mu2 value="100"/>
+      <kp value="1000000.0" />
+      <kd value="100.0" />
+      <slip1 value="0.5" />
+      <slip2 value="0.5" />
     <material>Gazebo/Red</material>
   </gazebo>
   <joint name="front_caster_joint" type="fixed">
-    <parent link="base_link"/>
+    <parent link="chassis"/>
     <child link="front_caster_link"/>
-    <origin xyz="0.0 -0.25 0.04" rpy="0 0 0"/>
+    <origin xyz="0.25 0.0 0.04" rpy="0 0 0"/>
     <mu1 value="0.001"/>
     <mu2 value="0.001"/>
@@ -123,7 +135,7 @@
   </gazebo>
   <joint name="back_caster_joint" type="fixed">
-    <parent link="base_link"/>
+    <parent link="chassis"/>
     <child link="back_caster_link"/>
-    <origin xyz="0.0 0.25 0.04" rpy="0 0 0"/>
+    <origin xyz="-0.25 0.0 0.04" rpy="0 0 0"/>
     <mu1 value="0.001"/>
     <mu2 value="0.001"/>
@@ -152,7 +164,7 @@
   </gazebo>
   <joint name="mount_joint" type="fixed">
-    <parent link="base_link"/>
+    <parent link="chassis"/>
     <child link="mount_link"/>
-    <origin xyz="0.0 -0.2 0.2" rpy="0.0 0.0 0.0"/>
+    <origin xyz="0.2 0.0 0.2" rpy="0.0 0.0 0.0"/>
   </joint>
   <link name="mount_link">
@@ -189,6 +201,6 @@
   </link>
   <joint name="camera_joint" type="fixed">
-    <origin xyz="0.0 -0.35 0.125" rpy="0 0 -1.57"/>
-    <parent link="base_link"/>
+    <origin xyz="0.35 0.0 0.125" rpy="0 0 0"/>
+    <parent link="chassis"/>
     <child link="camera_link"/>
   </joint>
@@ -204,5 +216,5 @@
     <material> Gazebo/Blue</material>
     <sensor type="camera" name="camera">
-      <update_rate>30.0</update_rate>
+      <update_rate>50.0</update_rate>
       <camera name="head">
           <horizontal_fov>1.3962634</horizontal_fov>
@@ -227,5 +239,5 @@
       <geometry>
         <cylinder radius="${lidar_radius}" length="${lidar_length}"/>
-        <!-- <mesh filename="package://round_bot/meshes/lds.stl" scale="0.001 0.001 0.001"/> -->
+        <!-- <mesh filename="package://round_bot/mesh/lds.stl" scale="0.001 0.001 0.001"/> -->
       </geometry>
       <material name="red">
@@ -236,5 +248,5 @@
       <geometry>
         <cylinder radius="${lidar_radius}" length="${lidar_length}"/>
-        <!-- <mesh filename="package://round_bot/meshes/lds.stl" scale="0.001 0.001 0.001"/> -->
+        <!-- <mesh filename="package://round_bot/mesh/lds.stl" scale="0.001 0.001 0.001"/> -->
       </geometry>
     </collision>
@@ -251,7 +263,7 @@
     <material> Gazebo/Red</material>
       <sensor name="gazebo_lidar" type="ray">
-      <always_on>true</always_on>
+      <pose> 0 0 0 0 0 0 </pose>
       <visualize>true</visualize>
-      <update_rate>30.0</update_rate>
+      <update_rate>50.0</update_rate>
       <ray>
         <scan>
@@ -259,12 +271,12 @@
             <samples>360</samples>
             <resolution>1.000000</resolution>
-            <min_angle>-3.14</min_angle>
-            <max_angle>3.14</max_angle>
+            <min_angle>-3.14159</min_angle>
+            <max_angle>3.14159</max_angle>
           </horizontal>
         </scan>
         <range>
-          <min>0.120000</min>
-          <max>3.5</max>
-          <resolution>0.015000</resolution>
+          <min>0.3</min>
+          <max>15.0</max>
+          <resolution>0.1</resolution>
         </range>
         <noise>
@@ -305,9 +317,9 @@
   <gazebo>
     <plugin name='diff_drive' filename='libgazebo_ros_diff_drive.so'>
-      <update_rate>30</update_rate>
+      <update_rate>50</update_rate>
       <left_joint>left_wheel_joint</left_joint>
-      <right_joint>right_wheel_joint</right_joint>\
+      <right_joint>right_wheel_joint</right_joint>
       <wheel_separation>0.50</wheel_separation>
-      <wheel_diameter>0.3</wheel_diameter>
+      <wheel_diameter>0.16</wheel_diameter>
       <max_wheel_torque>10</max_wheel_torque>
       <max_wheel_acceleration>1.0</max_wheel_acceleration>
@@ -315,7 +327,7 @@
       <publish_odom_tf>true</publish_odom_tf>
       <publish_wheel_tf>true</publish_wheel_tf>
-      <odometry_source>odom</odometry_source>
+      <odometry_source>1</odometry_source>
       <odometry_frame>odom</odometry_frame>
-      <robot_base_frame>base_footprint</robot_base_frame>
+      <robot_base_frame>base_link</robot_base_frame>
     </plugin>
   </gazebo>

Commit message: replaced MPPI with TEB planner

File: description/round_bot.urdf.xacro (robot description, xacro)
@@ -229,5 +229,4 @@
       <geometry>
         <cylinder radius="${lidar_radius}" length="${lidar_length}"/>
-        <!-- <mesh filename="package://round_bot/mesh/lds.stl" scale="0.001 0.001 0.001"/> -->
       </geometry>
       <material name="red">
@@ -238,5 +237,4 @@
       <geometry>
         <cylinder radius="${lidar_radius}" length="${lidar_length}"/>
-        <!-- <mesh filename="package://round_bot/mesh/lds.stl" scale="0.001 0.001 0.001"/> -->
       </geometry>
     </collision>
@@ -302,3 +300,32 @@
     </plugin>
   </gazebo>
+  <joint name="arm_base_joint" type="fixed">
+    <parent link="chassis"/>
+    <child link="arm_base"/>
+    <origin xyz="0.0 0.0 0.18" rpy="0.0 0.0 0.0"/>
+  </joint>
+  <link name="arm_base">
+    <visual>
+      <origin xyz="0.0 0.0 0.0" rpy="0.0 0.0 0.0"/>
+      <geometry>
+        <cylinder radius="0.1" length="0.015"/>
+      </geometry>
+      <material name ="Orange">
+        <color rgba = "1.0 0.0 0.0 1.0"/>
+      </material>
+    </visual>
+    <collision>
+      <origin xyz="0.0 0.0 0.0" rpy="0.0 0.0 0.0"/>
+      <geometry>
+        <cylinder radius="0.1" length="0.015"/>
+      </geometry>
+      <contact_coefficients mu1 = "1" mu2 = "1" kp = "1e+13.0" kd = "1.0"/>
+    </collision>
+    <xacro:inertial_chassis_cylinder chassis_mass="${chassis_mass}" chassis_length="${chassis_length}" chassis_radius="${chassis_radius}">
+      <origin xyz="0 0 0.12" rpy="0 0 0"/>
+    </xacro:inertial_chassis_cylinder>
+  </link>
+  <gazebo reference = "chassis">
+    <material>Gazebo/Red </material>
+  </gazebo>
 </robot>

Commit message: added stvl layer for 3d costmap

File: description/round_bot.urdf.xacro (robot description, xacro)
@@ -250,5 +250,5 @@
   <gazebo reference="lidar_link">
     <material> Gazebo/Red</material>
-      <sensor name="gazebo_lidar" type="ray">
+      <sensor name="block_laser_sensor" type="ray">
       <pose> 0 0 0 0 0 0 </pose>
       <visualize>true</visualize>
@@ -265,5 +265,5 @@
         <range>
           <min>0.3</min>
-          <max>5.0</max>
+          <max>2.5</max>
           <resolution>0.1</resolution>
         </range>
@@ -274,9 +274,10 @@
         </noise>
       </ray>
-      <plugin name="scan" filename="libgazebo_ros_ray_sensor.so">
+      <plugin name="gazebo_ros_block_laser_controller" filename="libgazebo_ros_ray_sensor.so">
         <ros>
-            <remapping>~/out:=scan</remapping>
+          <remapping>~/out:=scan</remapping>
         </ros>
         <output_type>sensor_msgs/LaserScan</output_type>
+        <!-- <output_type>sensor_msgs/PointCloud2</output_type> -->
         <frame_name>lidar_link</frame_name>
       </plugin>
@@ -300,5 +301,5 @@
     </plugin>
   </gazebo>
-  <joint name="arm_base_joint" type="fixed">
+  <!-- <joint name="arm_base_joint" type="fixed">
     <parent link="chassis"/>
     <child link="arm_base"/>
@@ -325,5 +326,5 @@
       <origin xyz="0 0 0.12" rpy="0 0 0"/>
     </xacro:inertial_chassis_cylinder>
-  </link>
+  </link> -->
   <gazebo reference = "chassis">
     <material>Gazebo/Red </material>
