Commit message: docker added and Plugins changed for gazebo Harmonic

File: description/round_bot.urdf.xacro (robot description, xacro)
@@ -2,5 +2,4 @@
 <robot xmlns:xacro="http://www.ros.org/wiki/xacro" name="round_bot">
   <xacro:include filename="$(find round_bot)/description/inertial_xacros.xacro"/>
-  <!-- <xacro:include filename="$(find round_bot)/description/ros2_control.xacro"/> -->
   <link name="base_footprint"/>
   <joint name="chassis_joint" type="fixed">
@@ -31,5 +30,5 @@
   </link>
   <gazebo reference = "chassis">
-    <material>Gazebo/Orange </material>
+    <material>Gazebo/Orange</material>
   </gazebo>
   <joint name="left_wheel_joint" type="continuous">
@@ -208,4 +207,5 @@
       <update_rate>50.0</update_rate>
       <camera name="head">
+        <camera_info_topic>camera/camera_info</camera_info_topic>
           <horizontal_fov>1.3962634</horizontal_fov>
           <image>
@@ -213,4 +213,5 @@
             <height>480</height>
             <format>R8G8B8</format>
+            <!-- <format>B8G8R8</format> -->
           </image>
           <clip>
@@ -219,8 +220,20 @@
           </clip>
       </camera>
-      <plugin name="camera_controller" filename="libgazebo_ros_camera.so">
+      <!-- <plugin name="camera_controller" filename="libgazebo_ros_camera.so">
         <alwaysOn>true</alwaysOn>
         <frameName>camera_link_optical</frameName>
-      </plugin>
+        <min_depth>0.1</min_depth>
+        <max_depth>100.0</max_depth>
+        <cameraName>head</cameraName>
+        <imageTopicName>/camera/image_raw</imageTopicName>
+        <cameraInfoTopicName>/camera/camera_info</cameraInfoTopicName>
+        <depthImageTopicName>/camera/depth/image_raw</depthImageTopicName>
+        <depthImageCameraInfoTopicName>/camera/depth/camera_info</depthImageCameraInfoTopicName>
+        <pointCloudTopicName>/camera/depth/points</pointCloudTopicName>
+        <pointCloudCutoff>0.05</pointCloudCutoff>
+        <pointCloudCutoffMax>8.0</pointCloudCutoffMax>
+      </plugin> -->
+      <topic>camera/image_raw</topic>
+      <gz_frame_id>camera_link_optical</gz_frame_id>
     </sensor>
   </gazebo>
@@ -250,9 +263,9 @@
   <gazebo reference="lidar_link">
     <material> Gazebo/Red</material>
-      <sensor name="block_laser_sensor" type="ray">
+      <sensor name="block_laser_sensor" type="gpu_lidar">
       <pose> 0 0 0 0 0 0 </pose>
       <visualize>true</visualize>
-      <update_rate>50.0</update_rate>
-      <ray>
+      <update_rate>10.0</update_rate>
+      <lidar>
         <scan>
           <horizontal>
@@ -265,5 +278,5 @@
         <range>
           <min>0.3</min>
-          <max>2.5</max>
+          <max>7.5</max>
           <resolution>0.1</resolution>
         </range>
@@ -273,60 +286,39 @@
           <stddev>0.01</stddev>
         </noise>
-      </ray>
-      <plugin name="gazebo_ros_block_laser_controller" filename="libgazebo_ros_ray_sensor.so">
+      </lidar>
+      <!-- <plugin name="gazebo_ros_block_laser_controller" filename="libgazebo_ros_ray_sensor.so">
         <ros>
           <remapping>~/out:=scan</remapping>
         </ros>
         <output_type>sensor_msgs/LaserScan</output_type>
-        <!-- <output_type>sensor_msgs/PointCloud2</output_type> -->
         <frame_name>lidar_link</frame_name>
-      </plugin>
+      </plugin> -->
+      <topic>scan</topic>
+      <gz_frame_id>lidar_link</gz_frame_id>
     </sensor>
   </gazebo>
   <gazebo>
-    <plugin name='diff_drive' filename='libgazebo_ros_diff_drive.so'>
+    <plugin name='gz::sim::systems::DiffDrive' filename='gz-sim-diff-drive-system'>
       <update_rate>50</update_rate>
       <left_joint>left_wheel_joint</left_joint>
       <right_joint>right_wheel_joint</right_joint>
       <wheel_separation>0.36</wheel_separation>
-      <wheel_diameter>0.16</wheel_diameter>
+      <wheel_radius>0.08</wheel_radius>
       <max_wheel_torque>10</max_wheel_torque>
-      <max_wheel_acceleration>1.0</max_wheel_acceleration>
-      <publish_odom>true</publish_odom>
-      <publish_odom_tf>true</publish_odom_tf>
-      <publish_wheel_tf>true</publish_wheel_tf>
-      <odometry_source>1</odometry_source>
-      <odometry_frame>odom</odometry_frame>
-      <robot_base_frame>base_footprint</robot_base_frame>
+      <max_linear_acceleration>10.0</max_linear_acceleration>
+      <max_angular_acceleration>3.0</max_angular_acceleration>
+      <frame_id>odom</frame_id>
+      <child_frame_id>base_footprint</child_frame_id>
+      <odom_topic>odom</odom_topic>
+      <odom_publisher_frequency>150</odom_publisher_frequency>
+      <tf_topic>/tf</tf_topic>
+      <topic>cmd_vel</topic>
     </plugin>
-  </gazebo>
-  <!-- <joint name="arm_base_joint" type="fixed">
-    <parent link="chassis"/>
-    <child link="arm_base"/>
-    <origin xyz="0.0 0.0 0.18" rpy="0.0 0.0 0.0"/>
-  </joint>
-  <link name="arm_base">
-    <visual>
-      <origin xyz="0.0 0.0 0.0" rpy="0.0 0.0 0.0"/>
-      <geometry>
-        <cylinder radius="0.1" length="0.015"/>
-      </geometry>
-      <material name ="Orange">
-        <color rgba = "1.0 0.0 0.0 1.0"/>
-      </material>
-    </visual>
-    <collision>
-      <origin xyz="0.0 0.0 0.0" rpy="0.0 0.0 0.0"/>
-      <geometry>
-        <cylinder radius="0.1" length="0.015"/>
-      </geometry>
-      <contact_coefficients mu1 = "1" mu2 = "1" kp = "1e+13.0" kd = "1.0"/>
-    </collision>
-    <xacro:inertial_chassis_cylinder chassis_mass="${chassis_mass}" chassis_length="${chassis_length}" chassis_radius="${chassis_radius}">
-      <origin xyz="0 0 0.12" rpy="0 0 0"/>
-    </xacro:inertial_chassis_cylinder>
-  </link> -->
-  <gazebo reference = "chassis">
-    <material>Gazebo/Red </material>
+    <plugin filename="gz-sim-joint-state-publisher-system"
+      name="gz::sim::systems::JointStatePublisher">
+      <topic>joint_states</topic>
+      <joint_name>left_wheel_joint</joint_name>
+      <joint_name>right_wheel_joint</joint_name>
+    </plugin>
   </gazebo>
 </robot>

Commit message: round_bot_in_outdoor

File: description/round_bot.urdf.xacro (robot description, xacro)
@@ -2,5 +2,4 @@
 <robot xmlns:xacro="http://www.ros.org/wiki/xacro" name="round_bot">
   <xacro:include filename="$(find round_bot)/description/inertial_xacros.xacro"/>
-  <xacro:property name="use_2d_lidar" value="true" />
   <link name="base_footprint"/>
   <joint name="chassis_joint" type="fixed">
@@ -53,4 +52,25 @@
       </geometry>
       <contact_coefficients mu1="1.0" mu2="1.0" kp="1000.0" kd="1.0"/>
+      <surface>
+        <friction>
+          <bullet>
+            <mu>1</mu>
+            <mu2>1</mu2>
+            <slip1>0.035</slip1>
+            <slip2>0</slip2>
+            <fdir1>0 0 1</fdir1>
+          </bullet>
+        </friction>
+        <contact>
+          <bullet>
+            <soft_cfm>0</soft_cfm>
+            <soft_erp>0.2</soft_erp>
+            <kp>1e+5</kp>
+            <kd>1</kd>
+            <max_vel>0.01</max_vel>
+            <min_depth>0.001</min_depth>
+          </bullet>
+        </contact>
+      </surface>
     </collision>
     <xacro:inertial_wheel_cylinder wheel_mass="${wheel_mass}" wheel_length="${wheel_length}" wheel_radius="${wheel_radius}">
@@ -81,4 +101,25 @@
       </geometry>
       <contact_coefficients mu1="1.0" mu2="1.0" kp="1000.0" kd="1.0"/>
+      <surface>
+        <friction>
+          <bullet>
+            <mu>1</mu>
+            <mu2>1</mu2>
+            <slip1>0.035</slip1>
+            <slip2>0</slip2>
+            <fdir1>0 0 1</fdir1>
+          </bullet>
+        </friction>
+        <contact>
+          <bullet>
+            <soft_cfm>0</soft_cfm>
+            <soft_erp>0.2</soft_erp>
+            <kp>1e+5</kp>
+            <kd>1</kd>
+            <max_vel>0.01</max_vel>
+            <min_depth>0.001</min_depth>
+          </bullet>
+        </contact>
+      </surface>
     </collision>
     <xacro:inertial_wheel_cylinder wheel_mass="${wheel_mass}" wheel_length="${wheel_length}" wheel_radius="${wheel_radius}">
@@ -110,4 +151,16 @@
       </geometry>
       <contact_coefficients mu="0" kp="1000.0" kd="1.0"/>
+      <surface>
+        <contact>
+          <bullet>
+            <soft_cfm>0</soft_cfm>
+            <soft_erp>0.2</soft_erp>
+            <kp>1e+5</kp>
+            <kd>1</kd>
+            <max_vel>0.01</max_vel>
+            <min_depth>0.001</min_depth>
+          </bullet>
+        </contact>
+      </surface>
     </collision>
     <xacro:inertial_sphere caster_mass="${caster_mass}" caster_radius="${caster_radius}">
@@ -139,4 +192,16 @@
       </geometry>
       <contact_coefficients mu="0" kp="1000.0" kd="1.0"/>
+      <surface>
+        <contact>
+          <bullet>
+            <soft_cfm>0</soft_cfm>
+            <soft_erp>0.2</soft_erp>
+            <kp>1e+5</kp>
+            <kd>1</kd>
+            <max_vel>0.01</max_vel>
+            <min_depth>0.001</min_depth>
+          </bullet>
+        </contact>
+      </surface>
     </collision>
     <xacro:inertial_sphere caster_mass="${caster_mass}" caster_radius="${caster_radius}">
@@ -147,30 +212,44 @@
     <material>Gazebo/Red</material>
   </gazebo>
-<!--  <joint name="mount_joint" type="fixed">
-    <parent link="chassis"/>
-    <child link="mount_link"/>
-    <origin xyz="0.15 0.0 0.18" rpy="0.0 0.0 0.0"/>
-  </joint>
-  <link name="mount_link">
-    <visual>
-      <geometry>
-        <cylinder radius="${mount_radius}" length="${mount_length}"/>
-      </geometry>
-      <material name="Black">
-        <color rgba="0.0 0.0 0.0 1.0"/>
-      </material>
-    </visual>
-    <collision>
-      <geometry>
-        <cylinder radius="${mount_radius}" length="${mount_length}"/>
-      </geometry>
-    </collision>
-    <xacro:inertial_mount_cylinder mount_mass="${mount_mass}" mount_length="${mount_length}" mount_radius="${mount_radius}">
-      <origin xyz="0 0 0" rpy="0 0 0"/>
-    </xacro:inertial_mount_cylinder>
-  </link>
-  <gazebo reference = "mount_link">
-    <material>Gazebo/Black</material>
-  </gazebo> -->
+  <joint name="gps_joint" type="fixed">
+    <origin xyz="0.0 0.0 0.17" rpy="0 0 0"/>
+    <parent link="chassis"/>
+    <child link = "gps_link"/>
+  </joint>
+  <link name="gps_link">
+    <visual>
+      <geometry>
+        <box size="0.03 0.03 0.01"/>
+      </geometry>
+      <material name="blue">
+        <color rgba="0 0 1 1"/>
+      </material>
+    </visual>
+  </link>
+  <gazebo reference = "gps_link">
+    <material>Gazebo/Blue</material>
+    <sensor name="navsat" type="navsat">
+      <always_on>true</always_on>
+      <update_rate>50</update_rate>
+      <topic>/navsat/fix</topic>
+      <gz_frame_id>gps_link</gz_frame_id>
+      <navsat>
+        <position_sensing>
+          <horizontal>
+            <noise type="gaussian">
+              <mean>0.0</mean>
+              <stddev>0.0</stddev>
+            </noise>
+          </horizontal>
+          <vertical>
+            <noise type="gaussian">
+              <mean>0.0</mean>
+              <stddev>0.0</stddev>
+            </noise>
+          </vertical>
+        </position_sensing>
+      </navsat>
+    </sensor>
+  </gazebo>
   <link name="imu_link">
     <visual>
@@ -183,15 +262,4 @@
       </material>
     </visual>
-    <collision>
-      <origin xyz="0 0 0.02" rpy="0 0 0"/>
-      <geometry>
-        <box size="0.03 0.03 0.02"/>
-      </geometry>
-    </collision>
-    <inertial>
-      <mass value="0.01"/>
-      <origin xyz="0 0 0.02" rpy="0 0 0"/>
-      <inertia ixx="1e-6" ixy="0" ixz="0" iyy="1e-6" iyz="0" izz="1e-6"/>
-    </inertial>
   </link>
   <joint name="imu_joint" type="fixed">
@@ -204,11 +272,62 @@
     <sensor name="imu_sensor" type="imu">
       <always_on>true</always_on>
-      <update_rate>100.0</update_rate>
+      <update_rate>50.0</update_rate>
       <visualize>true</visualize>
+      <gz_frame_id>imu_link</gz_frame_id>
       <topic>imu</topic>
-      <gz_frame_id>imu_link</gz_frame_id>
-      <plugin name="gz::sim::systems::Imu" filename="gz-sim-imu-system">
-        <topic>imu</topic>
-      </plugin>
+      <imu>
+      <angular_velocity>
+        <x>
+          <noise type="gaussian">
+            <mean>0.0</mean>
+            <stddev>2e-4</stddev>
+            <bias_mean>0.0000075</bias_mean>
+            <bias_stddev>0.0000008</bias_stddev>
+          </noise>
+        </x>
+        <y>
+          <noise type="gaussian">
+            <mean>0.0</mean>
+            <stddev>2e-4</stddev>
+            <bias_mean>0.0000075</bias_mean>
+            <bias_stddev>0.0000008</bias_stddev>
+          </noise>
+        </y>
+        <z>
+          <noise type="gaussian">
+            <mean>0.0</mean>
+            <stddev>2e-4</stddev>
+            <bias_mean>0.0000075</bias_mean>
+            <bias_stddev>0.0000008</bias_stddev>
+          </noise>
+        </z>
+      </angular_velocity>
+      <linear_acceleration>
+        <x>
+          <noise type="gaussian">
+            <mean>0.0</mean>
+            <stddev>1.7e-2</stddev>
+            <bias_mean>0.1</bias_mean>
+            <bias_stddev>0.001</bias_stddev>
+          </noise>
+        </x>
+        <y>
+          <noise type="gaussian">
+            <mean>0.0</mean>
+            <stddev>1.7e-2</stddev>
+            <bias_mean>0.1</bias_mean>
+            <bias_stddev>0.001</bias_stddev>
+          </noise>
+        </y>
+        <z>
+          <noise type="gaussian">
+            <mean>0.0</mean>
+            <stddev>1.7e-2</stddev>
+            <bias_mean>0.1</bias_mean>
+            <bias_stddev>0.001</bias_stddev>
+          </noise>
+        </z>
+      </linear_acceleration>
+    </imu>
     </sensor>
   </gazebo>
@@ -233,6 +352,5 @@
     <child link="camera_link_optical"/>
   </joint>
-  <link name="camera_link_optical">
-  </link>
+  <link name="camera_link_optical"/>
   <!-- camera -->
   <gazebo reference="camera_link">
@@ -283,76 +401,72 @@
   </joint>
   <!-- 2d lidar  -->
-  <xacro:if value="$(arg use_2d_lidar)">
-    <gazebo reference="lidar_link">
-      <material>Gazebo/Red</material>
-      <sensor name="hls_lfcd_lds" type="gpu_lidar">
-        <pose> 0 0 0 0 0 0 </pose>
-        <always_on>true</always_on>
-        <update_rate>30.0</update_rate>
-        <lidar>
-          <scan>
-            <horizontal>
-              <samples>360</samples>
-              <resolution>1.000000</resolution>
-              <min_angle>-3.14159</min_angle>
-              <max_angle>3.14159</max_angle>
-            </horizontal>
-          </scan>
-          <range>
-            <min>0.1</min>
-            <max>7.5</max>
+  <gazebo reference="lidar_link">
+    <material>Gazebo/Red</material>
+    <sensor name="hls_lfcd_lds" type="gpu_lidar">
+      <pose> 0 0 0 0 0 0 </pose>
+      <always_on>true</always_on>
+      <update_rate>30.0</update_rate>
+      <lidar>
+        <scan>
+          <horizontal>
+            <samples>360</samples>
+            <resolution>1.000000</resolution>
+            <min_angle>-3.14159</min_angle>
+            <max_angle>3.14159</max_angle>
+          </horizontal>
+        </scan>
+        <range>
+          <min>0.1</min>
+          <max>10.0</max>
+          <resolution>0.1</resolution>
+        </range>
+        <noise>
+          <type>gaussian</type>
+          <mean>0.0</mean>
+          <stddev>0.01</stddev>
+        </noise>
+      </lidar>
+      <topic>scan</topic>
+      <gz_frame_id>lidar_link</gz_frame_id>
+    </sensor>
+  </gazebo>
+  <!-- 3d lidar -->
+  <!-- <gazebo reference="lidar_link">
+    <material>Gazebo/Red</material>
+    <sensor name="block_laser_sensor" type="gpu_lidar">
+      <pose>0 0 0 0 0 0</pose>
+      <visualize>true</visualize>
+      <update_rate>30.0</update_rate>
+      <lidar>
+        <scan>
+          <horizontal>
+            <samples>180</samples>
+            <resolution>1.000000</resolution>
+            <min_angle>-3.14159</min_angle>
+            <max_angle>3.14159</max_angle>
+          </horizontal>
+          <vertical>
+            <samples>16</samples>
             <resolution>0.1</resolution>
-          </range>
-          <noise>
-            <type>gaussian</type>
-            <mean>0.0</mean>
-            <stddev>0.01</stddev>
-          </noise>
-        </lidar>
-        <topic>scan</topic>
-        <gz_frame_id>lidar_link</gz_frame_id>
-      </sensor>
-    </gazebo>
-  </xacro:if>
-  <!-- 3d lidar -->
-  <xacro:unless value="$(arg use_2d_lidar)">
-    <gazebo reference="lidar_link">
-      <material>Gazebo/Red</material>
-      <sensor name="block_laser_sensor" type="gpu_lidar">
-        <pose>0 0 0 0 0 0</pose>
-        <visualize>true</visualize>
-        <update_rate>30.0</update_rate>
-        <lidar>
-          <scan>
-            <horizontal>
-              <samples>180</samples>
-              <resolution>1.000000</resolution>
-              <min_angle>-3.14159</min_angle>
-              <max_angle>3.14159</max_angle>
-            </horizontal>
-            <vertical>
-              <samples>16</samples>
-              <resolution>0.1</resolution>
-              <min_angle>-0.2618</min_angle>
-              <max_angle>0.2618</max_angle>
-            </vertical>
-          </scan>
-          <range>
-            <min>0.5</min>
-            <max>7.5</max>
-            <resolution>0.1</resolution>
-          </range>
-          <point_cloud>true</point_cloud>
-          <noise>
-            <type>gaussian</type>
-            <mean>0.0</mean>
-            <stddev>0.01</stddev>
-          </noise>
-        </lidar>
-        <topic>velodyne_points</topic>
-        <gz_frame_id>lidar_link</gz_frame_id>
-      </sensor>
-    </gazebo>
-  </xacro:unless>
+            <min_angle>-0.2618</min_angle>
+            <max_angle>0.2618</max_angle>
+          </vertical>
+        </scan>
+        <range>
+          <min>0.5</min>
+          <max>7.5</max>
+          <resolution>0.1</resolution>
+        </range>
+        <point_cloud>true</point_cloud>
+        <noise>
+          <type>gaussian</type>
+          <mean>0.0</mean>
+          <stddev>0.01</stddev>
+        </noise>
+      </lidar>
+      <topic>velodyne_points</topic>
+      <gz_frame_id>lidar_link</gz_frame_id>
+    </sensor>
+  </gazebo> -->
   <gazebo>
     <plugin name='gz::sim::systems::DiffDrive' filename='gz-sim-diff-drive-system'>
@@ -361,11 +475,16 @@
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
Commit message: both planners and waypoint follower included

File: description/round_bot.urdf.xacro (robot description, xacro)
@@ -68,5 +68,5 @@
             <kp>1e+5</kp>
             <kd>1</kd>
-            <max_vel>0.01</max_vel>
+            <max_vel>1.0</max_vel>
             <min_depth>0.001</min_depth>
           </bullet>
@@ -117,5 +117,5 @@
             <kp>1e+5</kp>
             <kd>1</kd>
-            <max_vel>0.01</max_vel>
+            <max_vel>1.0</max_vel>
             <min_depth>0.001</min_depth>
           </bullet>
@@ -150,5 +150,5 @@
         <sphere radius="${caster_radius}"/>
       </geometry>
-      <contact_coefficients mu="0" kp="1000.0" kd="1.0"/>
+      <contact_coefficients mu="0.1" kp="1000.0" kd="1.0"/>
       <surface>
         <contact>
@@ -191,5 +191,5 @@
         <sphere radius="${caster_radius}"/>
       </geometry>
-      <contact_coefficients mu="0" kp="1000.0" kd="1.0"/>
+      <contact_coefficients mu="0.1" kp="1000.0" kd="1.0"/>
       <surface>
         <contact>
@@ -212,4 +212,30 @@
     <material>Gazebo/Red</material>
   </gazebo>
+  <!-- <joint name="mount_joint" type="fixed">
+    <parent link="chassis"/>
+    <child link="mount_link"/>
+    <origin xyz="0.15 0.0 0.18" rpy="0.0 0.0 0.0"/>
+  </joint>
+  <link name="mount_link">
+    <visual>
+      <geometry>
+        <cylinder radius="${mount_radius}" length="${mount_length}"/>
+      </geometry>
+      <material name="Black">
+        <color rgba="0.0 0.0 0.0 1.0"/>
+      </material>
+    </visual>
+    <collision>
+      <geometry>
+        <cylinder radius="${mount_radius}" length="${mount_length}"/>
+      </geometry>
+    </collision>
+    <xacro:inertial_mount_cylinder mount_mass="${mount_mass}" mount_length="${mount_length}" mount_radius="${mount_radius}">
+      <origin xyz="0 0 0" rpy="0 0 0"/>
+    </xacro:inertial_mount_cylinder>
+  </link>
+  <gazebo reference = "mount_link">
+    <material>Gazebo/Black</material>
+  </gazebo> -->
   <joint name="gps_joint" type="fixed">
     <origin xyz="0.0 0.0 0.17" rpy="0 0 0"/>
@@ -357,5 +383,5 @@
     <material> Gazebo/Blue</material>
     <sensor type="camera" name="camera">
-      <update_rate>10.0</update_rate>
+      <update_rate>50.0</update_rate>
       <camera name="head">
         <camera_info_topic>camera/camera_info</camera_info_topic>
@@ -406,5 +432,5 @@
       <pose> 0 0 0 0 0 0 </pose>
       <always_on>true</always_on>
-      <update_rate>30.0</update_rate>
+      <update_rate>50.0</update_rate>
       <lidar>
         <scan>
@@ -475,9 +501,9 @@
       <wheel_separation>0.36</wheel_separation>
       <wheel_radius>0.08</wheel_radius>
-      <max_linear_acceleration>1</max_linear_acceleration>
-      <min_linear_acceleration>-1</min_linear_acceleration>
-      <max_angular_acceleration>2</max_angular_acceleration>
-      <min_angular_acceleration>-2</min_angular_acceleration>
-      <max_linear_velocity>2.5</max_linear_velocity>
+      <max_linear_acceleration>10</max_linear_acceleration>
+      <min_linear_acceleration>-10</min_linear_acceleration>
+      <max_angular_acceleration>10</max_angular_acceleration>
+      <min_angular_acceleration>-10</min_angular_acceleration>
+      <max_linear_velocity>1.5</max_linear_velocity>
       <min_linear_velocity>0.0</min_linear_velocity>
       <max_angular_velocity>1.5</max_angular_velocity>
@@ -487,5 +513,6 @@
       <odom_topic>odom</odom_topic>
       <odom_publisher_frequency>50</odom_publisher_frequency>
-      <tf_topic>/tf</tf_topic>
+      <!-- comment this below one when you are using navigation, because we are letting ros to handle tf-->
+      <!-- <tf_topic>/tf</tf_topic> -->
       <topic>cmd_vel</topic>
     </plugin>
